File: PCB Diagrams/Audio Signal Injector.kicad_pcb (KiCad board)
At the start: 2 copper layers, 39.4 x 34.3 mm, 14 parts, among them J1 POWER, J2 POWER, J3 PROBE, U1 NE555P

Commit message: Adding project resources
Parts:
- C2: value 563 -> 100nF
- C3: value 104 -> 100nF
- R3: value 20K -> 100K
- RV1: value 5K -> 10K
- renumbered C4 to C1
Changed lines of the file:
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@@
 	(net 3 "C_VOLT")
 	(net 4 "OUTPUT")
-	(net 5 "Net-(C4-Pad2)")
+	(net 5 "Net-(C1-Pad2)")
 	(net 6 "VCC")
 	(net 7 "PROBE")
@@
 		(tags "C Disc series Radial pin pitch 5.00mm diameter 6mm width 2.5mm Capacitor")
 		(property "Reference" "C2"
-			(at 2.54 2.3 270)
-			(layer "F.SilkS")
-			(effects
-				(font
-					(size 1 1)
-					(thickness 0.15)
-				)
-			)
-		)
-		(property "Value" "563"
-			(at 2.5 0 90)
+			(at 2.667 0.0175 270)
+			(layer "F.SilkS")
+			(effects
+				(font
+					(size 1 1)
+					(thickness 0.15)
+				)
+			)
+		)
+		(property "Value" "100nF"
+			(at 2.667 2.0495 90)
 			(layer "F.Fab")
 			(effects
@@
 		(descr "C, Radial series, Radial, pin pitch=2.50mm, diameter=6.3mm, height=11mm, Non-Polar Electrolytic Capacitor")
 		(tags "C Radial series Radial pin pitch 2.50mm diameter 6.3mm height 11mm Non-Polar Electrolytic Capacitor")
-		(property "Reference" "C4"
+		(property "Reference" "C1"
 			(at 1.27 -2 0)
 			(layer "F.SilkS")
@@
 			(layers "*.Cu" "*.Mask")
 			(remove_unused_layers no)
-			(net 5 "Net-(C4-Pad2)")
+			(net 5 "Net-(C1-Pad2)")
 			(pintype "passive")
 		)
@@
 			)
 		)
-		(property "Value" "20K"
+		(property "Value" "100K"
 			(at 2.5 -0.7 0)
 			(layer "F.Fab")
@@
 		(tags "C Disc series Radial pin pitch 5.00mm diameter 6mm width 2.5mm Capacitor")
 		(property "Reference" "C3"
-			(at 5.04 2.54 0)
-			(layer "F.SilkS")
-			(effects
-				(font
-					(size 1 1)
-					(thickness 0.15)
-				)
-			)
-		)
-		(property "Value" "104"
-			(at 2.5 0 0)
+			(at 2.627 -0.127 0)
+			(layer "F.SilkS")
+			(effects
+				(font
+					(size 1 1)
+					(thickness 0.15)
+				)
+			)
+		)
+		(property "Value" "100nF"
+			(at 3.135 2.286 0)
 			(layer "F.Fab")
 			(effects
@@
 			)
 		)
-		(property "Value" "5K"
+		(property "Value" "10K"
 			(at -2.54 -2.54 0)
 			(layer "F.Fab")
@@
 			(remove_unused_layers no)
 			(roundrect_rratio 0.1388888889)
-			(net 5 "Net-(C4-Pad2)")
+			(net 5 "Net-(C1-Pad2)")
 			(pinfunction "1")
 			(pintype "passive")

Commit message: Adding folder 'Resources'
Parts:
- H1, H2: footprint MountingHole:MountingHole_2mm -> MountingHole:MountingHole_2.2mm_M2_ISO7380
- moved J3 1.27 mm to (171.4, 76.1)
Routing:
- net GND: track 0.00 -> 14.0 mm, vias 0 -> 2
- net PROBE: track 27.8 -> 29.0 mm
Changed lines of the file:
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@@
 	(footprint "TerminalBlock_Phoenix:TerminalBlock_Phoenix_PT-1,5-2-5.0-H_1x02_P5.00mm_Horizontal"
 		(layer "F.Cu")
-		(at 172.72 76.12 90)
+		(at 171.45 76.12 90)
 		(descr "Terminal Block Phoenix PT-1,5-2-5.0-H, 2 pins, pitch 5mm, size 10x9mm, drill diameter 1.3mm, pad diameter 2.6mm, http://www.mouser.com/ds/2/324/ItemDetail_1935161-922578.pdf, script-generated using https://gitlab.com/kicad/libraries/kicad-footprint-generator/-/tree/master/scripts/TerminalBlock_Phoenix")
 		(tags "THT Terminal Block Phoenix PT-1,5-2-5.0-H pitch 5mm size 10x9mm drill 1.3mm pad 2.6mm")
@@
 		(tags "Resistor Axial_DIN0207 series Axial Vertical pin pitch 2.54mm 0.25W = 1/4W length 6.3mm diameter 2.5mm")
 		(property "Reference" "R2"
-			(at 5.08 0 180)
+			(at 4.445 -1.27 180)
 			(layer "F.SilkS")
 			(effects
@@
 		)
 	)
-	(footprint "MountingHole:MountingHole_2mm"
+	(footprint "MountingHole:MountingHole_2.2mm_M2_ISO7380"
 		(layer "F.Cu")
 		(at 163.195 86.995)
-		(descr "Mounting Hole 2mm, no annular, generated by kicad-footprint-generator mountinghole.py")
-		(tags "mountinghole")
+		(descr "Mounting Hole 2.2mm, M2, no annular, generated by kicad-footprint-generator mountinghole.py")
+		(tags "mountinghole M2 ISO7380")
 		(property "Reference" "H2"
-			(at 0 -2.95 0)
+			(at 0 -2.7 0)
 			(layer "F.SilkS")
 			(hide yes)
@@
 		)
 		(property "Value" "MountingHole"
-			(at 0 2.95 0)
+			(at 0 2.7 0)
 			(layer "F.Fab")
 			(hide yes)
@@
 		(fp_circle
 			(center 0 0)
-			(end 2 0)
+			(end 1.75 0)
 			(stroke
 				(width 0.15)
@@
 		(fp_circle
 			(center 0 0)
-			(end 2.25 0)
+			(end 2 0)
 			(stroke
 				(width 0.05)
@@
 		(pad "" np_thru_hole circle
 			(at 0 0)
-			(size 2 2)
+			(size 2.2 2.2)
 			(drill 2)
 			(layers "*.Cu" "*.Mask")
@@
 		)
 	)
-	(footprint "MountingHole:MountingHole_2mm"
+	(footprint "MountingHole:MountingHole_2.2mm_M2_ISO7380"
 		(layer "F.Cu")
 		(at 144.78 78.74)
-		(descr "Mounting Hole 2mm, no annular, generated by kicad-footprint-generator mountinghole.py")
-		(tags "mountinghole")
+		(descr "Mounting Hole 2.2mm, M2, no annular, generated by kicad-footprint-generator mountinghole.py")
+		(tags "mountinghole M2 ISO7380")
 		(property "Reference" "H1"
-			(at 0 -2.95 0)
+			(at 0 -2.7 0)
 			(layer "F.SilkS")
 			(hide yes)
@@
 		)
 		(property "Value" "MountingHole"
-			(at 0 2.95 0)
+			(at 0 2.7 0)
 			(layer "F.Fab")
 			(hide yes)
@@
 		(fp_circle
 			(center 0 0)
-			(end 2 0)
+			(end 1.75 0)
 			(stroke
 				(width 0.15)
@@
 		(fp_circle
 			(center 0 0)
-			(end 2.25 0)
+			(end 2 0)
 			(stroke
 				(width 0.05)
@@
 		(pad "" np_thru_hole circle
 			(at 0 0)
-			(size 2 2)
+			(size 2.2 2.2)
 			(drill 2)
 			(layers "*.Cu" "*.Mask")
@@
 	)
 	(segment
+		(start 178.435 73.66)
+		(end 178.435 87.63)
+		(width 1.8)
+		(layer "F.Cu")
+		(net 1)
+	)
+	(via
+		(at 178.435 87.63)
+		(size 1.8)
+		(drill 1)
+		(layers "F.Cu" "B.Cu")
+		(free yes)
+		(net 1)
+	)
+	(via
+		(at 178.435 73.66)
+		(size 1.8)
+		(drill 1)
+		(layers "F.Cu" "B.Cu")
+		(free yes)
+		(net 1)
+	)
+	(segment
 		(start 156.21 71.12)
 		(end 165.095 71.12)
@@
 	)
 	(segment
+		(start 177.8 80.01)
+		(end 177.8 83.82)
+		(width 1.8)
+		(layer "B.Cu")
+		(net 7)
+	)
+	(segment
+		(start 171.45 90.17)
+		(end 171.45 98.44)
+		(width 1.8)
+		(layer "B.Cu")
+		(net 7)
+	)
+	(segment
+		(start 177.8 83.82)
+		(end 171.45 90.17)
+		(width 1.8)
+		(layer "B.Cu")
+		(net 7)
+	)
+	(segment
 		(start 173.91 76.12)
 		(end 177.8 80.01)
@@
 	)
 	(segment
-		(start 172.72 76.12)
+		(start 171.45 76.12)
 		(end 173.91 76.12)
-		(width 1.8)
-		(layer "B.Cu")
-		(net 7)
-	)
-	(segment
-		(start 171.45 90.17)
-		(end 171.45 98.44)
-		(width 1.8)
-		(layer "B.Cu")
-		(net 7)
-	)
-	(segment
-		(start 177.8 83.82)
-		(end 171.45 90.17)
-		(width 1.8)
-		(layer "B.Cu")
-		(net 7)
-	)
-	(segment
-		(start 177.8 80.01)
-		(end 177.8 83.82)
 		(width 1.8)
 		(layer "B.Cu")
@@
 		(hatch edge 0.5)
 		(connect_pads yes
-			(clearance 0.6)
+			(clearance 0.8)
 		)
 		(min_thickness 0.25)
