File: PCB Diagrams/Audio Signal Injector.kicad_sch (KiCad schematic)
At the start: 14 parts, among them J1 POWER, J2 POWER, J3 PROBE, U1 NE555P

Commit message: Adding project resources
Parts:
- C2: value 563 -> 100nF
- C3: value 104 -> 100nF
- R3: value 20K -> 100K
- RV1: value 5K -> 10K
- renumbered C4 to C1
Changed lines of the file:
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@@
 			)
 		)
-		(property "Value" "20K"
-			(at 193.802 99.06 90)
+		(property "Value" "100K"
+			(at 194.31 99.314 90)
 			(effects
 				(font
@@
 		(on_board yes)
 		(dnp no)
-		(property "Reference" "C4"
+		(property "Reference" "C1"
 			(at 182.626 81.28 90)
 			(effects
@@
 			(project ""
 				(path "/604830de-c4cb-461f-a5a7-02fc1d407f1c"
-					(reference "C4")
+					(reference "C1")
 					(unit 1)
 				)
@@
 			)
 		)
-		(property "Value" "104"
+		(property "Value" "100nF"
 			(at 180.34 75.438 90)
 			(effects
@@
 			)
 		)
-		(property "Value" "563"
-			(at 204.978 99.568 90)
+		(property "Value" "100nF"
+			(at 206.248 99.822 90)
 			(effects
 				(font
@@
 			)
 		)
-		(property "Value" "5K"
+		(property "Value" "10K"
 			(at 191.77 85.09 90)
 			(effects

Commit message: Adding folder 'Resources'
Parts:
- C2: value 100nF -> 56nF
- H1, H2: footprint MountingHole:MountingHole_2mm -> MountingHole:MountingHole_2.2mm_M2_ISO7380
- R3: value 100K -> 50K
Changed lines of the file:
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@@
 			)
 		)
-		(property "Value" "100K"
+		(property "Value" "50K"
 			(at 194.31 99.314 90)
 			(effects
@@
 			)
 		)
-		(property "Footprint" "MountingHole:MountingHole_2mm"
+		(property "Footprint" "MountingHole:MountingHole_2.2mm_M2_ISO7380"
 			(at 157.48 64.77 0)
 			(effects
@@
 			)
 		)
-		(property "Footprint" "MountingHole:MountingHole_2mm"
+		(property "Footprint" "MountingHole:MountingHole_2.2mm_M2_ISO7380"
 			(at 137.16 64.77 0)
 			(effects
@@
 			)
 		)
-		(property "Value" "100nF"
+		(property "Value" "56nF"
 			(at 206.248 99.822 90)
 			(effects
